Commit message: Updated URDF model and added revolute joint

File: urdf/scara.urdf (robot description, URDF)
Before this commit: robot myfirst, 1 links, 0 joints
Links:
- added link right_leg; visual box size=0.6 0.1 0.2
Joints:
- added joint base_to_right_leg: type continuous, parent base_link, child right_leg, origin xyz=0 -0.22 0.25

Commit message: First joint working in rviz

File: urdf/scara.urdf (robot description, URDF)
Before this commit: robot origins, 2 links, 1 joints
Links:
- removed link right_leg
- added link link1; visual cylinder length=${height1} radius=${width}
- link base_link: geometry visual cylinder length=0 radius=0
Joints:
- removed joint base_to_right_leg
- added joint base_to_link1: type continuous, parent base_link, child link1, origin xyz=0 0 0, axis 0 0 1

Commit message: Joint 2 in URDF model

File: urdf/scara.urdf (robot description, URDF)
Before this commit: robot scara, 2 links, 1 joints
Links:
- removed link base_link
- added link base; visual cylinder length=0 radius=0
- added link link2; visual cylinder length=${height2} radius=${width}
Joints:
- added joint link1_to_link2: type fixed, parent link1, child link2
- joint base_to_link1: parent base_link -> base

Commit message: second joint working on model

File: urdf/scara.urdf (robot description, URDF)
Before this commit: robot scara, 3 links, 2 joints
Links:
- added link link3; visual cylinder length=${height3} radius=${width}
Joints:
- added joint link2_to_link3: type continuous, parent link2, child link3, origin xyz=${height1} 0 0, axis 0 0 1
- joint link1_to_link2: origin (none) -> xyz=0 0 ${height1}

Commit message: URDF model working in rviz

File: urdf/scara.urdf (robot description, URDF)
Before this commit: robot scara, 4 links, 3 joints
Links:
- added link gripper_pole; visual cylinder length=0.2 radius=0.01
Joints:
- added joint gripper_extension: type prismatic, parent link3, child gripper_pole, origin xyz=${height3} 0 0 rpy=${PI} 0 0, axis 0 0 1, limit lower=0 upper=${prismatic_limit} effort=1000.0 velocity=0.5
- joint base_to_link1: limit (none) -> lower=${-PI} upper=${PI} effort=1000.0 velocity=0.5; type continuous -> revolute
- joint link2_to_link3: limit (none) -> lower=${-PI} upper=${PI} effort=1000.0 velocity=0.5; origin xyz=${height1} 0 0 -> xyz=${height2} 0 0; type continuous -> revolute
