Commit message: Working URDF model on gazebo

File: urdf/scara.xacro (robot description, xacro)
@@ -11,15 +11,4 @@
   <!-- Used for fixing robot to Gazebo 'base' -->
   <link name="world"/>
-  <link name="base">
-    <visual>
-      <geometry>
-        <cylinder length="0" radius="0"/>
-      </geometry>
-    </visual>
-  </link>
-  <joint name="fixed" type="fixed">
-    <parent link="world"/>
-    <child link="base"/>
-  </joint>
   <link name="link1">
     <collision>
@@ -45,5 +34,5 @@
   </link>
   <joint name="theta1" type="revolute">
-    <parent link="base"/>
+    <parent link="world"/>
     <child link="link1"/>
     <limit effort="1000.0" lower="${-PI}" upper="${PI}" velocity="0.5"/>

Commit message: Added joint publisher from gazebo. Ready to subscribe/publish to gazebo topics

File: urdf/scara.xacro (robot description, xacro)
@@ -7,4 +7,5 @@
   <xacro:property name="height" value="1" /> <!-- Link height -->
   <xacro:property name="prismatic_limit" value="1" /> <!-- Limit for prismatic joint -->
+  <xacro:property name="damping_coeff" value="0.7" /> <!-- Damping coefficient for joints -->
   <!-- Import all Gazebo-customization elements, including Gazebo colors -->
   <xacro:include filename="$(find rbe500_project)/urdf/scara.gazebo" />
@@ -39,4 +40,5 @@
     <axis xyz="0 0 1"/>
     <origin xyz="0 0 0"/>
+    <dynamics damping="${damping_coeff}"/>
   </joint>
   <link name="link2">
@@ -98,4 +100,5 @@
     <axis xyz="0 0 1"/>
     <origin xyz="${height} 0 0"/>
+    <dynamics damping="${damping_coeff}"/>
   </joint>
   <link name="gripper_pole">
@@ -127,4 +130,35 @@
     <axis xyz="0 0 1"/>
     <origin rpy="${PI} 0 0" xyz="${height} 0 0"/>
+    <dynamics damping="${damping_coeff}"/>
   </joint>
+  <transmission name="tran1">
+    <type>transmission_interface/SimpleTransmission</type>
+    <joint name="theta1">
+      <hardwareInterface>hardware_interface/EffortJointInterface</hardwareInterface>
+    </joint>
+    <actuator name="motor1">
+      <hardwareInterface>hardware_interface/EffortJointInterface</hardwareInterface>
+      <mechanicalReduction>1</mechanicalReduction>
+    </actuator>
+  </transmission>
+  <transmission name="tran2">
+    <type>transmission_interface/SimpleTransmission</type>
+    <joint name="theta2">
+      <hardwareInterface>hardware_interface/EffortJointInterface</hardwareInterface>
+    </joint>
+    <actuator name="motor2">
+      <hardwareInterface>hardware_interface/EffortJointInterface</hardwareInterface>
+      <mechanicalReduction>1</mechanicalReduction>
+    </actuator>
+  </transmission>
+  <transmission name="tran3">
+    <type>transmission_interface/SimpleTransmission</type>
+    <joint name="d3">
+      <hardwareInterface>hardware_interface/EffortJointInterface</hardwareInterface>
+    </joint>
+    <actuator name="motor3">
+      <hardwareInterface>hardware_interface/EffortJointInterface</hardwareInterface>
+      <mechanicalReduction>1</mechanicalReduction>
+    </actuator>
+  </transmission>
 </robot>

Commit message: Changed URDF model to work with boxes instead & early implementation of gravity compensation

File: urdf/scara.xacro (robot description, xacro)
@@ -6,4 +6,6 @@
   <xacro:property name="width" value="0.1" /> <!-- Square dimensions (widthxwidth) of beams -->
   <xacro:property name="height" value="1" /> <!-- Link height -->
+  <xacro:property name="width_pole" value="0.1" /> <!-- Square dimensions (widthxwidth) of beams -->
+  <xacro:property name="height_pole" value="0.1" /> <!-- Link height -->
   <xacro:property name="prismatic_limit" value="1" /> <!-- Limit for prismatic joint -->
   <xacro:property name="damping_coeff" value="0.7" /> <!-- Damping coefficient for joints -->
@@ -15,5 +17,5 @@
     <collision>
       <geometry>
-        <cylinder length="${height}" radius="${width}"/>
+        <box size="${width} ${width} ${height}"/>
       </geometry>
       <origin rpy="0 0 ${-PI}" xyz="0 0 ${height/2}"/>
@@ -21,5 +23,5 @@
     <visual>
       <geometry>
-        <cylinder length="${height}" radius="${width}"/>
+        <box size="${width} ${width} ${height}"/>
       </geometry>
       <origin rpy="0 0 ${-PI}" xyz="0 0 ${height/2}"/>
@@ -45,5 +47,5 @@
     <collision>
       <geometry>
-        <cylinder length="${height}" radius="${width}"/>
+        <box size="${width} ${width} ${height}"/>
       </geometry>
       <origin rpy="0 ${PI/2} 0" xyz="${height/2} 0 0"/>
@@ -51,5 +53,5 @@
     <visual>
       <geometry>
-        <cylinder length="${height}" radius="${width}"/>
+        <box size="${width} ${width} ${height}"/>
       </geometry>
       <material name="my_color">
@@ -75,5 +77,5 @@
     <collision>
       <geometry>
-        <cylinder length="${height}" radius="${width}"/>
+        <box size="${width} ${width} ${height}"/>
       </geometry>
       <origin rpy="0 ${PI/2} 0" xyz="${height/2} 0 0"/>
@@ -81,5 +83,5 @@
     <visual>
       <geometry>
-        <cylinder length="${height}" radius="${width}"/>
+        <box size="${width} ${width} ${height}"/>
       </geometry>
       <origin rpy="0 ${PI/2} 0" xyz="${height/2} 0 0"/>
@@ -105,5 +107,5 @@
     <collision>
       <geometry>
-        <cylinder length="0.2" radius="0.01"/>
+        <box size="${width_pole} ${width_pole} ${height_pole}"/>
       </geometry>
       <origin rpy="0 0 0 " xyz="0 0 0"/>
@@ -111,5 +113,5 @@
     <visual>
       <geometry>
-        <cylinder length="0.2" radius="0.01"/>
+        <box size="${width_pole} ${width_pole} ${height_pole}"/>
       </geometry>
       <origin rpy="0 0 0 " xyz="0 0 0"/>
@@ -119,7 +121,7 @@
       <mass value="${mass}"/>
       <inertia
-	  ixx="${mass / 12.0 * (width*width + height*height)}" ixy="0.0" ixz="0.0"
-	  iyy="${mass / 12.0 * (height*height + width*width)}" iyz="0.0"
-	  izz="${mass / 12.0 * (width*width + width*width)}"/>
+	  ixx="${mass / 12.0 * (width_pole*width_pole + height_pole*height_pole)}" ixy="0.0" ixz="0.0"
+	  iyy="${mass / 12.0 * (height_pole*height_pole + width_pole*width_pole)}" iyz="0.0"
+	  izz="${mass / 12.0 * (width_pole*width_pole + width_pole*width_pole)}"/>
     </inertial>
   </link>

Commit message: Implemented forward kinematics node.

File: urdf/scara.xacro (robot description, xacro)
@@ -6,4 +6,5 @@
   <xacro:property name="width" value="0.1" /> <!-- Square dimensions (widthxwidth) of beams -->
   <xacro:property name="height" value="1" /> <!-- Link height -->
+  <xacro:property name="mass_pole" value="0.01" /> <!-- arbitrary value for mass -->
   <xacro:property name="width_pole" value="0.1" /> <!-- Square dimensions (widthxwidth) of beams -->
   <xacro:property name="height_pole" value="0.1" /> <!-- Link height -->
@@ -119,5 +120,5 @@
     <inertial>
       <origin rpy="0 0 0 " xyz="0 0 0"/>
-      <mass value="${mass}"/>
+      <mass value="${mass_pole}"/>
       <inertia
 	  ixx="${mass / 12.0 * (width_pole*width_pole + height_pole*height_pole)}" ixy="0.0" ixz="0.0"

Commit message: Removed joint controller from sim

File: urdf/scara.xacro (robot description, xacro)
@@ -135,33 +135,3 @@
     <dynamics damping="${damping_coeff}"/>
   </joint>
-  <transmission name="tran1">
-    <type>transmission_interface/SimpleTransmission</type>
-    <joint name="theta1">
-      <hardwareInterface>hardware_interface/EffortJointInterface</hardwareInterface>
-    </joint>
-    <actuator name="motor1">
-      <hardwareInterface>hardware_interface/EffortJointInterface</hardwareInterface>
-      <mechanicalReduction>1</mechanicalReduction>
-    </actuator>
-  </transmission>
-  <transmission name="tran2">
-    <type>transmission_interface/SimpleTransmission</type>
-    <joint name="theta2">
-      <hardwareInterface>hardware_interface/EffortJointInterface</hardwareInterface>
-    </joint>
-    <actuator name="motor2">
-      <hardwareInterface>hardware_interface/EffortJointInterface</hardwareInterface>
-      <mechanicalReduction>1</mechanicalReduction>
-    </actuator>
-  </transmission>
-  <transmission name="tran3">
-    <type>transmission_interface/SimpleTransmission</type>
-    <joint name="d3">
-      <hardwareInterface>hardware_interface/EffortJointInterface</hardwareInterface>
-    </joint>
-    <actuator name="motor3">
-      <hardwareInterface>hardware_interface/EffortJointInterface</hardwareInterface>
-      <mechanicalReduction>1</mechanicalReduction>
-    </actuator>
-  </transmission>
 </robot>

Commit message: Reimplemented functionality to drive joints to given position via gazebo model config proxy

File: urdf/scara.xacro (robot description, xacro)
@@ -6,5 +6,5 @@
   <xacro:property name="width" value="0.1" /> <!-- Square dimensions (widthxwidth) of beams -->
   <xacro:property name="height" value="1" /> <!-- Link height -->
-  <xacro:property name="mass_pole" value="0.01" /> <!-- arbitrary value for mass -->
+  <xacro:property name="mass_pole" value="0.1" /> <!-- arbitrary value for mass -->
   <xacro:property name="width_pole" value="0.1" /> <!-- Square dimensions (widthxwidth) of beams -->
   <xacro:property name="height_pole" value="0.1" /> <!-- Link height -->

Commit message: Fixed joints theta1 and theta2, no longer launching ford kin node to avoid errors.

File: urdf/scara.xacro (robot description, xacro)
@@ -37,5 +37,5 @@
     </inertial>
   </link>
-  <joint name="theta1" type="revolute">
+  <joint name="theta1" type="fixed">
     <parent link="world"/>
     <child link="link1"/>
@@ -97,5 +97,5 @@
     </inertial>
   </link>
-  <joint name="theta2" type="revolute">
+  <joint name="theta2" type="fixed">
     <parent link="link2"/>
     <child link="link3"/>

Commit message: Implemented PD controller

File: urdf/scara.xacro (robot description, xacro)
@@ -6,5 +6,5 @@
   <xacro:property name="width" value="0.1" /> <!-- Square dimensions (widthxwidth) of beams -->
   <xacro:property name="height" value="1" /> <!-- Link height -->
-  <xacro:property name="mass_pole" value="0.1" /> <!-- arbitrary value for mass -->
+  <xacro:property name="mass_pole" value="0.01" /> <!-- arbitrary value for mass -->
   <xacro:property name="width_pole" value="0.1" /> <!-- Square dimensions (widthxwidth) of beams -->
   <xacro:property name="height_pole" value="0.1" /> <!-- Link height -->

Commit message: changes to ROM of d3 + improvements to PD controller + disabling gravity for EE

File: urdf/scara.xacro (robot description, xacro)
@@ -6,5 +6,5 @@
   <xacro:property name="width" value="0.1" /> <!-- Square dimensions (widthxwidth) of beams -->
   <xacro:property name="height" value="1" /> <!-- Link height -->
-  <xacro:property name="mass_pole" value="0.01" /> <!-- arbitrary value for mass -->
+  <xacro:property name="mass_pole" value="0.1" /> <!-- arbitrary value for mass -->
   <xacro:property name="width_pole" value="0.1" /> <!-- Square dimensions (widthxwidth) of beams -->
   <xacro:property name="height_pole" value="0.1" /> <!-- Link height -->
@@ -130,8 +130,11 @@
     <parent link="link3"/>
     <child link="gripper_pole"/>
-    <limit effort="1000.0" lower="0" upper="${prismatic_limit}" velocity="0.5"/>
+    <limit effort="1000.0" lower="${-prismatic_limit}" upper="${prismatic_limit}" velocity="0.5"/>
     <axis xyz="0 0 1"/>
     <origin rpy="${PI} 0 0" xyz="${height} 0 0"/>
     <dynamics damping="${damping_coeff}"/>
   </joint>
+  <gazebo reference="gripper_pole">
+    <turnGravityOff>true</turnGravityOff>
+  </gazebo>
 </robot>

Commit message: Added PD controller support for theta1 and theta2 joints, also added publisher for joint velocities at a rate of 0.1 seconds

File: urdf/scara.xacro (robot description, xacro)
@@ -37,5 +37,5 @@
     </inertial>
   </link>
-  <joint name="theta1" type="fixed">
+  <joint name="theta1" type="revolute">
     <parent link="world"/>
     <child link="link1"/>
@@ -97,5 +97,5 @@
     </inertial>
   </link>
-  <joint name="theta2" type="fixed">
+  <joint name="theta2" type="revolute">
     <parent link="link2"/>
     <child link="link3"/>
@@ -135,4 +135,10 @@
     <dynamics damping="${damping_coeff}"/>
   </joint>
+  <gazebo reference="theta1">
+    <turnGravityOff>true</turnGravityOff>
+  </gazebo>
+  <gazebo reference="theta2">
+    <turnGravityOff>true</turnGravityOff>
+  </gazebo>
   <gazebo reference="gripper_pole">
     <turnGravityOff>true</turnGravityOff>
